File: RC-710/Schematic/Schematic.kicad_sch (KiCad schematic)
At the start: 65 parts, among them K1 Fujitsu_FTR-LYAA005x, Q1 NPN, Q2 NPN, SW1 ON/OFF, SW2 LEARN, U1 LM358, Y1 Crystal

Commit message: Schematic: Improved layout
Signed-off-by: Patrick Pedersen <ctx.xda@gmail.com>
Parts:
- removed R25: R, symbol Device:R
- added R13: R, symbol Device:R
- added U2: ~, symbol RC-710:Blob_IC
- Y1: value Crystal -> 455kHZ
Connections:
- net Blob IC PB LEARN: now also U2. (VCC)
- net Blob IC PB ON/OFF: now also U2. (VCC)
- net Blob IC REF CLK A: now also U2. (VCC)
- net Blob IC REF CLK B: now also U2. (VCC)
- net Blob IC SIGNAL: now also U2. (VCC)
- net GND: now also U2. (VCC)
- net V1: no longer C11.1, C16.2, D10.2 (A), D13.1 (K), R16.1, R23.1, R7.1, U1.8 (V+)
- net Blob IC RST?: no longer names the net of TP2.1
- net Blob IC RST?: now also R13.1, U2. (VCC)
- net Blob IC UNKNOWN: no longer names the net of TP1.1
- net Blob IC UNKNOWN: now also U2. (VCC)
- net Blob IC VCC? renamed +3V0
- net +3V0: now also R13.2, U2. (VCC)
- net ~{Blob IC RELAY} renamed Blob IC RELAY
- net Blob IC RELAY: now also U2. (VCC)
- new net +5V: C11.1, C16.2, D10.2 (A), D13.1 (K), R16.1, R23.1, R7.1, U1.8 (V+)
Other:
- note added: "Caution: May contain mistakes!"
- note added: "Handles device logic and RF signal processing"
- note added: "IC + Demod. Clock"
- note added: "IC Power"
- note added: "Mandolyn RC-710 Remote Power Socket"
- note added: "Misc"
- note added: "Power"
- note added: "Push Buttons"
- note added: "RF Circuit"
- note added: "Relay Switching"
- note added: "Schematic reverse engineered by: Patrick Pedersen"
- note added: "This device uses an unisolated power supply. This effectively means that all low voltages here are FLOATING AT MAINS VOLTAGE! Merely touching any GND terminal while the device is plugged in WILL SHOCK YOU with up to 325V!"
- note added: "Unknown Blob IC"
- note added: "WARNING: ELECTRICAL HAZARD"
- note added: "When testing the device it is highly recommended to connect a bench supply with 24VDC at betweem the recitfier output (C13) and GND. This eliminates the electrical hazard."
- note added: "~3V"
- moved on the sheet: C1, C10, C14, C15, C17, C18, C19, C2, C3, C4, C5, C6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

Commit message: README: Added text
Signed-off-by: Patrick Pedersen <ctx.xda@gmail.com>
Parts:
- Q1: value NPN -> KSP10
- Q2: value NPN -> C9014
Other:
- note added: "Bleeder"
- moved on the sheet: C13, R19
Changed lines of the file:
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@@
 	(wire
 		(pts
+			(xy 71.12 34.29) (xy 71.12 43.18)
+		)
+		(stroke
+			(width 0)
+			(type default)
+		)
+	)
+	(wire
+		(pts
 			(xy 152.4 231.14) (xy 152.4 247.65)
 		)
@@
 	(wire
 		(pts
-			(xy 55.88 43.18) (xy 55.88 49.53)
-		)
-		(stroke
-			(width 0)
-			(type default)
-		)
-	)
-	(wire
-		(pts
 			(xy 137.16 171.45) (xy 137.16 186.69)
 		)
@@
 	(wire
 		(pts
-			(xy 71.12 43.18) (xy 71.12 49.53)
-		)
-		(stroke
-			(width 0)
-			(type default)
-		)
-	)
-	(wire
-		(pts
 			(xy 195.58 168.91) (xy 204.47 168.91)
 		)
@@
 	(wire
 		(pts
-			(xy 67.31 43.18) (xy 71.12 43.18)
+			(xy 67.31 34.29) (xy 71.12 34.29)
 		)
 		(stroke
@@
 	(wire
 		(pts
-			(xy 55.88 49.53) (xy 59.69 49.53)
+			(xy 55.88 43.18) (xy 59.69 43.18)
 		)
 		(stroke
@@
 	(wire
 		(pts
+			(xy 55.88 34.29) (xy 55.88 43.18)
+		)
+		(stroke
+			(width 0)
+			(type default)
+		)
+	)
+	(wire
+		(pts
 			(xy 50.8 168.91) (xy 59.69 168.91)
 		)
@@
 	(wire
 		(pts
-			(xy 67.31 49.53) (xy 71.12 49.53)
+			(xy 67.31 43.18) (xy 71.12 43.18)
 		)
 		(stroke
@@
 	(wire
 		(pts
-			(xy 55.88 43.18) (xy 59.69 43.18)
+			(xy 55.88 34.29) (xy 59.69 34.29)
 		)
 		(stroke
@@
 		)
 	)
+	(text "Bleeder"
+		(exclude_from_sim no)
+		(at 63.5 36.83 0)
+		(effects
+			(font
+				(size 1.27 1.27)
+			)
+		)
+	)
 	(global_label "Blob IC RELAY"
 		(shape input)
@@
 		(dnp no)
 		(property "Reference" "Q1"
-			(at 181.102 189.992 90)
+			(at 181.61 189.992 90)
 			(effects
 				(font
@@
 			)
 		)
-		(property "Value" "NPN"
-			(at 182.372 192.532 90)
+		(property "Value" "KSP10"
+			(at 183.642 192.532 90)
 			(effects
 				(font
@@
 		(at 229.87 83.82 0)
 		(unit 1)
-		(exclude_from_sim no)
+		(exclude_from_sim yes)
 		(in_bom no)
 		(on_board no)
@@
 			)
 		)
-		(property "Sim.Enable" "0"
-			(at 229.87 83.82 0)
-			(effects
-				(font
-					(size 1.27 1.27)
-				)
-				(hide yes)
-			)
-		)
 		(instances
 			(project ""
@@
 	(symbol
 		(lib_id "Device:C")
-		(at 63.5 49.53 90)
+		(at 63.5 43.18 90)
 		(unit 1)
 		(exclude_from_sim no)
@@
 		(dnp no)
 		(property "Reference" "C13"
-			(at 63.5 54.61 90)
+			(at 63.5 48.26 90)
 			(effects
 				(font
@@
 		)
 		(property "Value" "0.22uF"
-			(at 63.5 57.15 90)
+			(at 63.5 50.8 90)
 			(effects
 				(font
@@
 		)
 		(property "Footprint" ""
-			(at 67.31 48.5648 0)
+			(at 67.31 42.2148 0)
 			(effects
 				(font
@@
 		)
 		(property "Datasheet" "~"
-			(at 63.5 49.53 0)
+			(at 63.5 43.18 0)
 			(effects
 				(font
@@
 		)
 		(property "Description" "Unpolarized capacitor"
-			(at 63.5 49.53 0)
+			(at 63.5 43.18 0)
 			(effects
 				(font
@@
 	(symbol
 		(lib_id "Device:R")
-		(at 63.5 43.18 90)
+		(at 63.5 34.29 90)
 		(unit 1)
 		(exclude_from_sim no)
@@
 		(fields_autoplaced yes)
 		(property "Reference" "R19"
-			(at 63.5 36.83 90)
+			(at 63.5 27.94 90)
 			(effects
 				(font
@@
 		)
 		(property "Value" "1M"
-			(at 63.5 39.37 90)
+			(at 63.5 30.48 90)
 			(effects
 				(font
@@
 		)
 		(property "Footprint" ""
-			(at 63.5 44.958 90)
+			(at 63.5 36.068 90)
 			(effects
 				(font
@@
 		)
 		(property "Datasheet" "~"
-			(at 63.5 43.18 0)
+			(at 63.5 34.29 0)
 			(effects
 				(font
@@
 		)
 		(property "Description" "Resistor"
-			(at 63.5 43.18 0)
+			(at 63.5 34.29 0)
 			(effects
 				(font
@@
 			)
 		)
-		(property "Value" "NPN"
+		(property "Value" "C9014"
 			(at 190.5 59.6899 0)
 			(effects

Commit message: README: Updated + Schematic: Minor correction
Signed-off-by: Patrick Pedersen <ctx.xda@gmail.com>
Other:
- note added: "IC Clock"
- note removed: "IC + Demod. Clock"
Changed lines of the file:
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@@
 		)
 	)
-	(text "IC + Demod. Clock"
+	(text "IC Clock"
 		(exclude_from_sim no)
 		(at 104.14 97.79 0)
